File: STM32F405RGT6_BlackPill/MCU.kicad_sch (KiCad schematic)
At the start: 40 parts, among them J100 Conn_01x04, J101 Conn_02x15_Odd_Even, J102 Conn_02x10_Odd_Even, J103 Conn_01x02, U100 STM32F405RGTx, Y1 32768Hz, Y100 25Mhz

Commit message: Production files JLCPCB
Parts:
- C114, C115: Manufacturer TDK Corporation -> Samsung Electro-Mechanics; Manufacturer Product Number C2012X7R1C225K125AB -> CL21B225KAFNNNE
- D103: Manufacturer Würth Elektronik -> Hubei KENTO Elec; Manufacturer Product Number 150060GS75000 -> KT-0603R
- L100: Manufacturer Johanson Technology Inc. -> Murata Electronics; Manufacturer Product Number LRC0402CJ10NGV001T -> LQG15HS10NJ02D
- R100, R101, R102, R107: Manufacturer Samsung Electro-Mechanics -> UNI-ROYAL(Uniroyal Elec); Manufacturer Product Number RC1005F103CS -> 0402WGF1002TCE
- R103, R104, R105, R106: Manufacturer Panasonic Electronic Components -> UNI-ROYAL(Uniroyal Elec); Manufacturer Product Number ERJ-2GEJ470X -> 0402WGF470JTCE
- R108: Manufacturer Panasonic Electronic Components -> UNI-ROYAL(Uniroyal Elec); Manufacturer Product Number ERA-2AEB512X -> 0402WGF5101TCE
- Y100: Manufacturer Abracon LLC -> YXC Crystal Oscillators; Manufacturer Product Number ASE-25.000MHZ-L-C-T -> OT322525MJBA4SL
- Y101: renamed from Y1; Manufacturer Abracon LLC -> YXC Crystal Oscillators; Manufacturer Product Number ASEK-32.768KHZ-L-R-T -> OK2EL89CJI-111YLC-32.768K
Changed lines of the file:
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@@
 			)
 		)
-		(property "Manufacturer" "TDK Corporation"
+		(property "Manufacturer" "Samsung Electro-Mechanics"
 			(at 87.63 146.05 0)
 			(effects
@@
 			)
 		)
-		(property "Manufacturer Product Number" "C2012X7R1C225K125AB"
+		(property "Manufacturer Product Number" "CL21B225KAFNNNE"
 			(at 87.63 146.05 0)
 			(effects
@@
 			)
 		)
-		(property "Manufacturer" "Samsung Electro-Mechanics"
+		(property "Manufacturer" "UNI-ROYAL(Uniroyal Elec)"
 			(at 52.07 40.64 0)
 			(effects
@@
 			)
 		)
-		(property "Manufacturer Product Number" "RC1005F103CS"
+		(property "Manufacturer Product Number" "0402WGF1002TCE"
 			(at 52.07 40.64 0)
 			(effects
@@
 			)
 		)
-		(property "Manufacturer" "Würth Elektronik"
+		(property "Manufacturer" "Hubei KENTO Elec"
 			(at 62.23 128.27 0)
 			(effects
@@
 			)
 		)
-		(property "Manufacturer Product Number" "150060GS75000"
+		(property "Manufacturer Product Number" "KT-0603R"
 			(at 62.23 128.27 0)
 			(effects
@@
 			)
 		)
-		(property "Manufacturer" "Samsung Electro-Mechanics"
+		(property "Manufacturer" "UNI-ROYAL(Uniroyal Elec)"
 			(at 36.83 41.91 0)
 			(effects
@@
 			)
 		)
-		(property "Manufacturer Product Number" "RC1005F103CS"
+		(property "Manufacturer Product Number" "0402WGF1002TCE"
 			(at 36.83 41.91 0)
 			(effects
@@
 		(on_board yes)
 		(dnp no)
-		(property "Reference" "Y1"
+		(property "Reference" "Y101"
 			(at 244.602 27.94 0)
 			(effects
@@
 			)
 		)
-		(property "Manufacturer" "Abracon LLC"
+		(property "Manufacturer" "YXC Crystal Oscillators"
 			(at 242.57 33.02 0)
 			(effects
@@
 			)
 		)
-		(property "Manufacturer Product Number" "ASEK-32.768KHZ-L-R-T"
+		(property "Manufacturer Product Number" "OK2EL89CJI-111YLC-32.768K"
 			(at 242.57 33.02 0)
 			(effects
@@
 			(project "STM32F405RGT6_BlackPill"
 				(path "/cae5b0ba-cc42-4347-bdfb-a704c1b808ff/dd7f6eda-dc83-4b84-a9a2-d4778c0007f8"
-					(reference "Y1")
+					(reference "Y101")
 					(unit 1)
 				)
@@
 	)
 	(symbol
+		(lib_name "BlackPillLibrary:SW_PUSH_6mm_H5mm")
 		(lib_id "BlackPillLibrary:SW_PUSH_6mm_H5mm")
 		(at 29.21 119.38 270)
@@
 	)
 	(symbol
+		(lib_name "BlackPillLibrary:SW_PUSH_6mm_H5mm")
 		(lib_id "BlackPillLibrary:SW_PUSH_6mm_H5mm")
 		(at 96.52 35.56 270)
@@
 			)
 		)
-		(property "Manufacturer" "Abracon LLC"
+		(property "Manufacturer" "YXC Crystal Oscillators"
 			(at 196.85 30.48 0)
 			(effects
@@
 			)
 		)
-		(property "Manufacturer Product Number" "ASE-25.000MHZ-L-C-T"
+		(property "Manufacturer Product Number" "OT322525MJBA4SL"
 			(at 196.85 30.48 0)
 			(effects
@@
 			)
 		)
-		(property "Manufacturer" "TDK Corporation"
+		(property "Manufacturer" "Samsung Electro-Mechanics"
 			(at 95.25 146.05 0)
 			(effects
@@
 			)
 		)
-		(property "Manufacturer Product Number" "C2012X7R1C225K125AB"
+		(property "Manufacturer Product Number" "CL21B225KAFNNNE"
 			(at 95.25 146.05 0)
 			(effects
@@
 			)
 		)
-		(property "Manufacturer" "Panasonic Electronic Components"
+		(property "Manufacturer" "UNI-ROYAL(Uniroyal Elec)"
 			(at 252.73 26.67 0)
 			(effects
@@
 			)
 		)
-		(property "Manufacturer Product Number" "ERJ-2GEJ470X"
+		(property "Manufacturer Product Number" "0402WGF470JTCE"
 			(at 252.73 26.67 0)
 			(effects
@@
 			)
 		)
-		(property "Manufacturer" "Panasonic Electronic Components"
+		(property "Manufacturer" "UNI-ROYAL(Uniroyal Elec)"
 			(at 59.69 78.74 0)
 			(effects
@@
 			)
 		)
-		(property "Manufacturer Product Number" "ERJ-2GEJ470X"
+		(property "Manufacturer Product Number" "0402WGF470JTCE"
 			(at 59.69 78.74 0)
 			(effects
@@
 			)
 		)
-		(property "Manufacturer" "Panasonic Electronic Components"
+		(property "Manufacturer" "UNI-ROYAL(Uniroyal Elec)"
 			(at 208.28 24.13 0)
 			(effects
@@
 			)
 		)
-		(property "Manufacturer Product Number" "ERJ-2GEJ470X"
+		(property "Manufacturer Product Number" "0402WGF470JTCE"
 			(at 208.28 24.13 0)
 			(effects
@@
 	)
 	(symbol
+		(lib_name "BlackPillLibrary:SW_PUSH_6mm_H5mm")
 		(lib_id "BlackPillLibrary:SW_PUSH_6mm_H5mm")
 		(at 27.94 33.02 270)
@@
 			)
 		)
-		(property "Manufacturer" "Johanson Technology Inc."
+		(property "Manufacturer" "Murata Electronics"
 			(at 170.18 27.94 0)
 			(effects
@@
 			)
 		)
-		(property "Manufacturer Product Number" "LRC0402CJ10NGV001T"
+		(property "Manufacturer Product Number" "LQG15HS10NJ02D"
 			(at 170.18 27.94 0)
 			(effects
@@
 			)
 		)
-		(property "Manufacturer" "Samsung Electro-Mechanics"
+		(property "Manufacturer" "UNI-ROYAL(Uniroyal Elec)"
 			(at 38.1 128.27 0)
 			(effects
@@
 			)
 		)
-		(property "Manufacturer Product Number" "RC1005F103CS"
+		(property "Manufacturer Product Number" "0402WGF1002TCE"
 			(at 38.1 128.27 0)
 			(effects
@@
 			)
 		)
-		(property "Manufacturer" "Panasonic Electronic Components"
+		(property "Manufacturer" "UNI-ROYAL(Uniroyal Elec)"
 			(at 59.69 76.2 0)
 			(effects
@@
 			)
 		)
-		(property "Manufacturer Product Number" "ERJ-2GEJ470X"
+		(property "Manufacturer Product Number" "0402WGF470JTCE"
 			(at 59.69 76.2 0)
 			(effects
@@
 			)
 		)
-		(property "Manufacturer" "Samsung Electro-Mechanics"
+		(property "Manufacturer" "UNI-ROYAL(Uniroyal Elec)"
 			(at 82.55 29.21 0)
 			(effects
@@
 			)
 		)
-		(property "Manufacturer Product Number" "RC1005F103CS"
+		(property "Manufacturer Product Number" "0402WGF1002TCE"
 			(at 82.55 29.21 0)
 			(effects
@@
 			)
 		)
-		(property "Manufacturer" "Panasonic Electronic Components"
+		(property "Manufacturer" "UNI-ROYAL(Uniroyal Elec)"
 			(at 62.23 118.11 0)
 			(effects
@@
 			)
 		)
-		(property "Manufacturer Product Number" "ERA-2AEB512X"
+		(property "Manufacturer Product Number" "0402WGF5101TCE"
 			(at 62.23 118.11 0)
 			(effects
