File: STM32F405RGT6_BlackPill/usb.kicad_sch (KiCad schematic)
At the start: 6 parts, among them J2 USB_C_Receptacle_USB2.0_16P, U2 USBLC6-2SC6

Commit message: First version of the scheme
Changed lines of the file:
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@@
 		(dnp no)
 		(property "Reference" "U2"
-			(at 149.86 46.99 0)
+			(at 146.558 51.054 0)
 			(effects
 				(font

Commit message: Essential part of the BOM fill
Parts:
- removed L2: CMF3216F-900-2P-T, symbol Device:EMI_Filter_LL_1423
- added U201: ACM2012-900-2P-T001, BlackPill:SMT_0-2P-T001_TDK, symbol BlackPillLibrary:ACM2012-900-2P-T001
- C200: renamed from C16; LCSC link https://www.lcsc.com/product-detail/Multilayer-Ceramic-Capa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 -> (none); Manufacturer Samwha Capacitor -> (none); Manufacturer Part Number CS1005X7R104K500NR -> (none)
- U200: renamed from U2; DigiKey Part Number (none) -> 497-5235-6-ND; LCSC link https://www.lcsc.com/product-detail/ESD-and-Surge-Protectio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 -> (none); Manufacturer TECH PUBLIC -> STMicroelectronics; Manufacturer Part Number USBLC6-2SC6 -> (none); Manufacturer Product Number (none) -> USBLC6-2SC6
- renumbered J2 to J200, R8 to R200, R9 to R201
Connections:
- net USB_CMC_D+: now also U201.2
- net USB_CMC_D-: now also U201.1
- net USB_D+: now also U201.3
- net USB_D-: now also U201.4
Changed lines of the file:
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@@
-	(wire
-		(pts
-			(xy 73.66 58.42) (xy 64.77 58.42)
-		)
-		(stroke
-			(width 0)
-			(type default)
-		)
-	)
 	(wire
 		(pts
@@
 	(wire
 		(pts
+			(xy 64.77 52.07) (xy 67.31 52.07)
+		)
+		(stroke
+			(width 0)
+			(type default)
+		)
+	)
+	(wire
+		(pts
+			(xy 102.87 44.45) (xy 116.84 44.45)
+		)
+		(stroke
+			(width 0)
+			(type default)
+		)
+	)
+	(wire
+		(pts
 			(xy 194.31 57.15) (xy 185.42 57.15)
 		)
@@
 	(wire
 		(pts
-			(xy 102.87 58.42) (xy 83.82 58.42)
-		)
-		(stroke
-			(width 0)
-			(type default)
-		)
-	)
-	(wire
-		(pts
 			(xy 215.9 36.83) (xy 218.44 36.83)
 		)
@@
 	(wire
 		(pts
-			(xy 102.87 53.34) (xy 83.82 53.34)
-		)
-		(stroke
-			(width 0)
-			(type default)
-		)
-	)
-	(wire
-		(pts
 			(xy 215.9 57.15) (xy 215.9 54.61)
 		)
@@
 	(wire
 		(pts
+			(xy 102.87 52.07) (xy 116.84 52.07)
+		)
+		(stroke
+			(width 0)
+			(type default)
+		)
+	)
+	(wire
+		(pts
 			(xy 121.92 58.42) (xy 139.7 58.42)
 		)
@@
 	(wire
 		(pts
+			(xy 64.77 44.45) (xy 67.31 44.45)
+		)
+		(stroke
+			(width 0)
+			(type default)
+		)
+	)
+	(wire
+		(pts
 			(xy 233.68 74.93) (xy 233.68 80.01)
 		)
@@
 		(pts
 			(xy 149.86 58.42) (xy 167.64 58.42)
-		)
-		(stroke
-			(width 0)
-			(type default)
-		)
-	)
-	(wire
-		(pts
-			(xy 73.66 53.34) (xy 64.77 53.34)
 		)
 		(stroke
@@
 	(text "Common-Mode Choke Impedance: 90R"
 		(exclude_from_sim no)
-		(at 55.118 64.516 0)
+		(at 67.818 59.182 0)
 		(effects
 			(font
@@
 	)
 	(label "USB_CMC_D-"
-		(at 102.87 58.42 180)
+		(at 116.84 52.07 180)
 		(fields_autoplaced yes)
 		(effects
@@
 	)
 	(label "USB_CMC_D+"
-		(at 102.87 53.34 180)
+		(at 116.84 44.45 180)
 		(fields_autoplaced yes)
 		(effects
@@
 	(global_label "USB_D-"
 		(shape input)
-		(at 64.77 58.42 180)
+		(at 64.77 52.07 180)
 		(fields_autoplaced yes)
 		(effects
@@
 		)
 		(property "Intersheetrefs" "${INTERSHEET_REFS}"
-			(at 54.1648 58.42 0)
+			(at 54.1648 52.07 0)
 			(effects
 				(font
@@
 	(global_label "USB_D+"
 		(shape input)
-		(at 64.77 53.34 180)
+		(at 64.77 44.45 180)
 		(fields_autoplaced yes)
 		(effects
@@
 		)
 		(property "Intersheetrefs" "${INTERSHEET_REFS}"
-			(at 54.1648 53.34 0)
+			(at 54.1648 44.45 0)
 			(effects
 				(font
@@
 	)
 	(symbol
-		(lib_id "Device:EMI_Filter_LL_1423")
-		(at 78.74 55.88 0)
-		(mirror y)
+		(lib_id "BlackPillLibrary:ACM2012-900-2P-T001")
+		(at 107.95 52.07 180)
 		(unit 1)
 		(exclude_from_sim no)
@@
 		(on_board yes)
 		(dnp no)
-		(property "Reference" "L2"
-			(at 78.74 60.96 0)
-			(effects
-				(font
-					(size 1.27 1.27)
-				)
-			)
-		)
-		(property "Value" "CMF3216F-900-2P-T"
-			(at 78.74 50.8 0)
-			(effects
-				(font
-					(size 1.27 1.27)
-				)
-			)
-		)
-		(property "Footprint" ""
-			(at 78.74 62.23 0)
-			(effects
-				(font
-					(size 1.27 1.27)
-				)
-				(hide yes)
-			)
-		)
-		(property "Datasheet" "~"
-			(at 78.74 54.864 90)
-			(effects
-				(font
-					(size 1.27 1.27)
+		(fields_autoplaced yes)
+		(property "Reference" "U201"
+			(at 85.09 39.37 0)
+			(effects
+				(font
+					(size 1.524 1.524)
+				)
+			)
+		)
+		(property "Value" "ACM2012-900-2P-T001"
+			(at 85.09 41.91 0)
+			(effects
+				(font
+					(size 1.524 1.524)
+				)
+			)
+		)
+		(property "Footprint" "BlackPill:SMT_0-2P-T001_TDK"
+			(at 107.95 52.07 0)
+			(effects
+				(font
+					(size 1.27 1.27)
+					(italic yes)
+				)
+				(hide yes)
+			)
+		)
+		(property "Datasheet" "ACM2012-900-2P-T001"
+			(at 107.95 52.07 0)
+			(effects
+				(font
+					(size 1.27 1.27)
+					(italic yes)
 				)
 				(hide yes)
@@
 		)
 		(property "Description" ""
-			(at 78.74 55.88 0)
-			(effects
-				(font
-					(size 1.27 1.27)
-				)
-				(hide yes)
-			)
+			(at 107.95 52.07 0)
+			(effects
+				(font
+					(size 1.27 1.27)
+				)
+				(hide yes)
+			)
+		)
+		(pin "3"
+		)
+		(pin "2"
+		)
+		(pin "4"
 		)
 		(pin "1"
 		)
-		(pin "2"
-		)
-		(pin "3"
-		)
-		(pin "4"
-		)
 		(instances
-			(project "STM32F405RGT6_BlackPill"
+			(project ""
 				(path "/cae5b0ba-cc42-4347-bdfb-a704c1b808ff/eb317edf-4a76-4641-bee6-7756ac9721d3"
-					(reference "L2")
+					(reference "U201")
 					(unit 1)
 				)
@@
 		(on_board yes)
 		(dnp no)
-		(property "Reference" "U2"
+		(property "Reference" "U200"
 			(at 146.558 51.054 0)
 			(effects
@@
 			)
 		)
-		(property "LCSC Parrt #" ""
+		(property "Manufacturer" "STMicroelectronics"
 			(at 144.78 55.88 0)
 			(effects
@@
 			)
 		)
-		(property "LCSC link" "https://www.lcsc.com/product-detail/ESD-and-Surge-Protection-TVS-ESD_TECH-PUBLIC-USBLC6-2SC6_C2827654.html"
+		(property "DigiKey Part Number" "497-5235-6-ND"
 			(at 144.78 55.88 0)
 			(effects
@@
 			)
 		)
-		(property "Manufacturer" "TECH PUBLIC"
-			(at 144.78 55.88 0)
-			(effects
-				(font
-					(size 1.27 1.27)
-				)
-				(hide yes)
-			)
-		)
-		(property "Manufacturer Part Number" "USBLC6-2SC6"
+		(property "Manufacturer Product Number" "USBLC6-2SC6"
 			(at 144.78 55.88 0)
 			(effects
@@
 			(project "STM32F405RGT6_BlackPill"
 				(path "/cae5b0ba-cc42-4347-bdfb-a704c1b808ff/eb317edf-4a76-4641-bee6-7756ac9721d3"
-					(reference "U2")
+					(reference "U200")
 					(unit 1)
 				)
@@
 		(on_board yes)
 		(dnp no)
-		(property "Reference" "J2"
+		(property "Reference" "J200"
 			(at 240.03 31.496 0)
 			(effects
@@
 		)
 		(property "Description" "USB 2.0-only 16P Type-C Receptacle connector"
+			(at 233.68 52.07 0)
+			(effects
+				(font
+					(size 1.27 1.27)
+				)
+				(hide yes)
+			)
+		)
+		(property "DigiKey Part Number" ""
 			(at 233.68 52.07 0)
 			(effects
@@
 			(project "STM32F405RGT6_BlackPill"
 				(path "/cae5b0ba-cc42-4347-bdfb-a704c1b808ff/eb317edf-4a76-4641-bee6-7756ac9721d3"
-					(reference "J2")
+					(reference "J200")
 					(unit 1)
 				)
@@
 		(dnp no)
 		(fields_autoplaced yes)
-		(property "Reference" "R8"
+		(property "Reference" "R200"
 			(at 187.96 48.2599 0)
 			(effects
@@
 		)
 		(property "Description" "Resistor"
+			(at 185.42 49.53 0)
+			(effects
+				(font
+					(size 1.27 1.27)
+				)
+				(hide yes)
+			)
+		)
+		(property "DigiKey Part Number" ""
 			(at 185.42 49.53 0)
 			(effects
@@
 			(project "STM32F405RGT6_BlackPill"
 				(path "/cae5b0ba-cc42-4347-bdfb-a704c1b808ff/eb317edf-4a76-4641-bee6-7756ac9721d3"
-					(reference "R8")
+					(reference "R200")
 					(unit 1)
 				)
@@
 		(on_board yes)
 		(dnp no)
-		(property "Reference" "C16"
+		(property "Reference" "C200"
 			(at 130.81 39.37 90)
 			(effects
@@
 			)
 		)
-		(property "LCSC link" "https://www.lcsc.com/product-detail/Multilayer-Ceramic-Capacitors-MLCC-SMD-SMT_Samwha-Capacitor-CS1005X7R104K500NR_C513772.html"
+		(property "Manufacturer" ""
 			(at 133.35 43.18 0)
 			(effects
@@
 			)
 		)
-		(property "Manufacturer" "Samwha Capacitor"
-			(at 133.35 43.18 0)
-			(effects
-				(font
-					(size 1.27 1.27)
-				)
-				(hide yes)
-			)
-		)
-		(property "Manufacturer Part Number" "CS1005X7R104K500NR"
+		(property "DigiKey Part Number" ""
 			(at 133.35 43.18 0)
 			(effects
@@
 			(project "STM32F405RGT6_BlackPill"
 				(path "/cae5b0ba-cc42-4347-bdfb-a704c1b808ff/eb317edf-4a76-4641-bee6-7756ac9721d3"
-					(reference "C16")
+					(reference "C200")
 					(unit 1)
 				)
@@
 		(dnp no)
 		(fields_autoplaced yes)
-		(property "Reference" "R9"
+		(property "Reference" "R201"
 			(at 196.85 48.2599 0)
 			(effects
@@
 		)
 		(property "Description" "Resistor"
+			(at 194.31 49.53 0)
+			(effects
+				(font
+					(size 1.27 1.27)
+				)
+				(hide yes)
+			)
+		)
+		(property "DigiKey Part Number" ""
 			(at 194.31 49.53 0)
 			(effects
@@
 			(project "STM32F405RGT6_BlackPill"
 				(path "/cae5b0ba-cc42-4347-bdfb-a704c1b808ff/eb317edf-4a76-4641-bee6-7756ac9721d3"
-					(reference "R9")
+					(reference "R201")
 					(unit 1)
 				)

Commit message: BOM table fill
Parts:
- C200: DigiKey Part Number (none) -> 1276-1002-6-ND; Manufacturer (none) -> Samsung Electro-Mechanics; Manufacturer Product Number (none) -> CL05B104KP5NNNC
- J200: DigiKey Part Number (none) -> 664-12402012E212ADKR-ND; Manufacturer (none) -> Amphenol ICC (Commercial Products); Manufacturer Product Number (none) -> 12402012E212A
- R200, R201: DigiKey Part Number (none) -> P5.1KDCDKR-ND; Manufacturer (none) -> Panasonic Electronic Components; Manufacturer Product Number (none) -> ERA-2AEB512X
- U201: DigiKey Part Number (none) -> 445-15969-6-ND; Manufacturer (none) -> TDK Corporation; Manufacturer Product Number (none) -> ACM2012-900-2P-T001
Changed lines of the file:
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@@
+			)
+		)
+		(property "DigiKey Part Number" "445-15969-6-ND"
+			(at 107.95 52.07 0)
+			(effects
+				(font
+					(size 1.27 1.27)
+				)
+				(hide yes)
+			)
+		)
+		(property "Manufacturer" "TDK Corporation"
+			(at 107.95 52.07 0)
+			(effects
+				(font
+					(size 1.27 1.27)
+				)
+				(hide yes)
+			)
+		)
+		(property "Manufacturer Product Number" "ACM2012-900-2P-T001"
+			(at 107.95 52.07 0)
+			(effects
+				(font
+					(size 1.27 1.27)
+				)
+				(hide yes)
 			)
 		)
@@
 			)
 		)
-		(property "DigiKey Part Number" ""
+		(property "DigiKey Part Number" "664-12402012E212ADKR-ND"
+			(at 233.68 52.07 0)
+			(effects
+				(font
+					(size 1.27 1.27)
+				)
+				(hide yes)
+			)
+		)
+		(property "Manufacturer" "Amphenol ICC (Commercial Products)"
+			(at 233.68 52.07 0)
+			(effects
+				(font
+					(size 1.27 1.27)
+				)
+				(hide yes)
+			)
+		)
+		(property "Manufacturer Product Number" "12402012E212A"
 			(at 233.68 52.07 0)
 			(effects
@@
 			)
 		)
-		(property "DigiKey Part Number" ""
+		(property "DigiKey Part Number" "P5.1KDCDKR-ND"
+			(at 185.42 49.53 0)
+			(effects
+				(font
+					(size 1.27 1.27)
+				)
+				(hide yes)
+			)
+		)
+		(property "Manufacturer" "Panasonic Electronic Components"
+			(at 185.42 49.53 0)
+			(effects
+				(font
+					(size 1.27 1.27)
+				)
+				(hide yes)
+			)
+		)
+		(property "Manufacturer Product Number" "ERA-2AEB512X"
 			(at 185.42 49.53 0)
 			(effects
@@
 			)
 		)
-		(property "Manufacturer" ""
+		(property "Manufacturer" "Samsung Electro-Mechanics"
 			(at 133.35 43.18 0)
 			(effects
@@
 			)
 		)
-		(property "DigiKey Part Number" ""
+		(property "DigiKey Part Number" "1276-1002-6-ND"
+			(at 133.35 43.18 0)
+			(effects
+				(font
+					(size 1.27 1.27)
+				)
+				(hide yes)
+			)
+		)
+		(property "Manufacturer Product Number" "CL05B104KP5NNNC"
 			(at 133.35 43.18 0)
 			(effects
@@
 			)
 		)
-		(property "DigiKey Part Number" ""
+		(property "DigiKey Part Number" "P5.1KDCDKR-ND"
 			(at 194.31 49.53 0)
 			(effects
+				(font
+					(size 1.27 1.27)
+				)
+				(hide yes)
+			)
+		)
+		(property "Manufacturer" "Panasonic Electronic Components"
+			(at 194.31 49.53 0)
+			(effects
+				(font
+					(size 1.27 1.27)
+				)
+				(hide yes)
+			)
+		)
+		(property "Manufacturer Product Number" "ERA-2AEB512X"
+			(at 194.31 49.53 0)
+			(effects

Commit message: Production files JLCPCB
Parts:
- J200: Manufacturer Amphenol ICC (Commercial Products) -> Korean Hroparts Elec; Manufacturer Product Number 12402012E212A -> TYPE-C-31-M-12
- R200, R201: Manufacturer Panasonic Electronic Components -> UNI-ROYAL(Uniroyal Elec); Manufacturer Product Number ERA-2AEB512X -> 0402WGF5101TCE
Changed lines of the file:
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@@
 			)
 		)
-		(property "Manufacturer" "Amphenol ICC (Commercial Products)"
+		(property "Manufacturer" "Korean Hroparts Elec"
 			(at 233.68 52.07 0)
 			(effects
@@
 			)
 		)
-		(property "Manufacturer Product Number" "12402012E212A"
+		(property "Manufacturer Product Number" "TYPE-C-31-M-12"
 			(at 233.68 52.07 0)
 			(effects
@@
 			)
 		)
-		(property "Manufacturer" "Panasonic Electronic Components"
+		(property "Manufacturer" "UNI-ROYAL(Uniroyal Elec)"
 			(at 185.42 49.53 0)
 			(effects
@@
 			)
 		)
-		(property "Manufacturer Product Number" "ERA-2AEB512X"
+		(property "Manufacturer Product Number" "0402WGF5101TCE"
 			(at 185.42 49.53 0)
 			(effects
@@
 			)
 		)
-		(property "Manufacturer" "Panasonic Electronic Components"
+		(property "Manufacturer" "UNI-ROYAL(Uniroyal Elec)"
 			(at 194.31 49.53 0)
 			(effects
@@
 			)
 		)
-		(property "Manufacturer Product Number" "ERA-2AEB512X"
+		(property "Manufacturer Product Number" "0402WGF5101TCE"
 			(at 194.31 49.53 0)
 			(effects
